Commit message: added depth odometry testing launcher

File: urdf/stereo_camera.urdf.xacro (robot description, xacro)
@@ -23,15 +23,15 @@
     </link>
     <!-- Left camera -->
-    <link name="left_camera_frame"/>
+    <link name="left_camera_optical_frame"/>
     <joint name="left_camera_joint" type="fixed">
       <parent link="camera_link"/>
-      <child link="left_camera_frame"/>
+      <child link="left_camera_optical_frame"/>
       <origin xyz="${-baseline/2} 0 0" rpy="0 0 0"/>
     </joint>
     <!-- Right camera -->
-    <link name="right_camera_frame"/>
+    <link name="right_camera_optical_frame"/>
     <joint name="right_camera_joint" type="fixed">
       <parent link="camera_link"/>
-      <child link="right_camera_frame"/>
+      <child link="right_camera_optical_frame"/>
       <origin xyz="${baseline/2} 0 0" rpy="0 0 0"/>
     </joint>

Commit message: point cloud update

File: urdf/stereo_camera.urdf.xacro (robot description, xacro)
@@ -2,5 +2,5 @@
 <robot xmlns:xacro="http://www.ros.org/wiki/xacro" name="stereo_camera">
   <xacro:property name="M_PI" value="3.1415926535897931" />
-  <xacro:property name="baseline" value="0.06" /> <!-- 60mm -->
+  <xacro:property name="baseline" value="0.0152" /> <!-- 60mm -->
   <xacro:property name="camera_width" value="0.085" /> <!-- 85mm -->
   <xacro:property name="camera_height" value="0.024" /> <!-- 24mm -->

Commit message: small yaml changes and camera height implementation

File: urdf/stereo_camera.urdf.xacro (robot description, xacro)
@@ -1,10 +1,13 @@
 <?xml version="1.0"?>
 <robot xmlns:xacro="http://www.ros.org/wiki/xacro" name="stereo_camera">
+  <!-- Constants -->
   <xacro:property name="M_PI" value="3.1415926535897931" />
   <xacro:property name="baseline" value="0.0152" /> <!-- 60mm -->
   <xacro:property name="camera_width" value="0.085" /> <!-- 85mm -->
   <xacro:property name="camera_height" value="0.024" /> <!-- 24mm -->
+  <!-- Parameter for camera and IMU height above ground -->
+  <xacro:property name="camera_height_above_ground" value="0.7"/> <!-- adjust this value (meters) -->
   <xacro:macro name="stereo_camera_macro" params="parent *origin">
-    <!-- Base link -->
+    <!-- Base camera box -->
     <link name="camera_link">
       <visual>
@@ -22,5 +25,5 @@
       </collision>
     </link>
-    <!-- Left camera -->
+    <!-- Left camera optical frame -->
     <link name="left_camera_optical_frame"/>
     <joint name="left_camera_joint" type="fixed">
@@ -29,5 +32,5 @@
       <origin xyz="${-baseline/2} 0 0" rpy="0 0 0"/>
     </joint>
-    <!-- Right camera -->
+    <!-- Right camera optical frame -->
     <link name="right_camera_optical_frame"/>
     <joint name="right_camera_joint" type="fixed">
@@ -36,5 +39,5 @@
       <origin xyz="${baseline/2} 0 0" rpy="0 0 0"/>
     </joint>
-    <!-- IMU -->
+    <!-- IMU link -->
     <link name="imu_link"/>
     <joint name="imu_joint" type="fixed">
@@ -43,14 +46,15 @@
       <origin xyz="0 0 0" rpy="0 0 0"/>
     </joint>
-    <!-- Mount to parent -->
+    <!-- Mount camera to parent (base_link), offset vertically -->
     <joint name="camera_mount_joint" type="fixed">
       <xacro:insert_block name="origin"/>
       <parent link="${parent}"/>
       <child link="camera_link"/>
+      <origin xyz="0 0 ${camera_height_above_ground}" rpy="0 0 0"/>
     </joint>
   </xacro:macro>
   <!-- Create base link -->
   <link name="base_link"/>
-  <!-- Instantiate the stereo camera -->
+  <!-- Instantiate stereo camera -->
   <xacro:stereo_camera_macro parent="base_link">
     <origin xyz="0 0 0" rpy="0 0 0"/>

Commit message: more tuning

File: urdf/stereo_camera.urdf.xacro (robot description, xacro)
@@ -29,6 +29,7 @@
     <joint name="left_camera_joint" type="fixed">
       <parent link="camera_link"/>
-      <child link="left_camera_optical_frame"/>
-      <origin xyz="${-baseline/2} 0 0" rpy="0 0 0"/>
+      <child  link="left_camera_optical_frame"/>
+      <!-- left camera sits +Y -->
+      <origin xyz="0 ${baseline/2} 0" rpy="0 0 0"/>
     </joint>
     <!-- Right camera optical frame -->
@@ -36,6 +37,7 @@
     <joint name="right_camera_joint" type="fixed">
       <parent link="camera_link"/>
-      <child link="right_camera_optical_frame"/>
-      <origin xyz="${baseline/2} 0 0" rpy="0 0 0"/>
+      <child  link="right_camera_optical_frame"/>
+      <!-- right camera sits –Y -->
+      <origin xyz="0 ${-baseline/2} 0" rpy="0 0 0"/>
     </joint>
     <!-- IMU link -->

Commit message: odometry works

File: urdf/stereo_camera.urdf.xacro (robot description, xacro)
@@ -1,13 +1,10 @@
 <?xml version="1.0"?>
 <robot xmlns:xacro="http://www.ros.org/wiki/xacro" name="stereo_camera">
-  <!-- Constants -->
   <xacro:property name="M_PI" value="3.1415926535897931" />
   <xacro:property name="baseline" value="0.0152" /> <!-- 60mm -->
   <xacro:property name="camera_width" value="0.085" /> <!-- 85mm -->
   <xacro:property name="camera_height" value="0.024" /> <!-- 24mm -->
-  <!-- Parameter for camera and IMU height above ground -->
-  <xacro:property name="camera_height_above_ground" value="0.7"/> <!-- adjust this value (meters) -->
   <xacro:macro name="stereo_camera_macro" params="parent *origin">
-    <!-- Base camera box -->
+    <!-- Base link -->
     <link name="camera_link">
       <visual>
@@ -25,21 +22,19 @@
       </collision>
     </link>
-    <!-- Left camera optical frame -->
+    <!-- Left camera -->
     <link name="left_camera_optical_frame"/>
     <joint name="left_camera_joint" type="fixed">
       <parent link="camera_link"/>
-      <child  link="left_camera_optical_frame"/>
-      <!-- left camera sits +Y -->
-      <origin xyz="0 ${baseline/2} 0" rpy="0 0 0"/>
+      <child link="left_camera_optical_frame"/>
+      <origin xyz="${-baseline/2} 0 0" rpy="-1.57079632679 0 -1.57079632679"/>
     </joint>
-    <!-- Right camera optical frame -->
+    <!-- Right camera -->
     <link name="right_camera_optical_frame"/>
     <joint name="right_camera_joint" type="fixed">
       <parent link="camera_link"/>
-      <child  link="right_camera_optical_frame"/>
-      <!-- right camera sits –Y -->
-      <origin xyz="0 ${-baseline/2} 0" rpy="0 0 0"/>
+      <child link="right_camera_optical_frame"/>
+      <origin xyz="${baseline/2} 0 0" rpy="-1.57079632679 0 -1.57079632679"/>
     </joint>
-    <!-- IMU link -->
+    <!-- IMU -->
     <link name="imu_link"/>
     <joint name="imu_joint" type="fixed">
@@ -48,15 +43,14 @@
       <origin xyz="0 0 0" rpy="0 0 0"/>
     </joint>
-    <!-- Mount camera to parent (base_link), offset vertically -->
+    <!-- Mount to parent -->
     <joint name="camera_mount_joint" type="fixed">
       <xacro:insert_block name="origin"/>
       <parent link="${parent}"/>
       <child link="camera_link"/>
-      <origin xyz="0 0 ${camera_height_above_ground}" rpy="0 0 0"/>
     </joint>
   </xacro:macro>
   <!-- Create base link -->
   <link name="base_link"/>
-  <!-- Instantiate stereo camera -->
+  <!-- Instantiate the stereo camera -->
   <xacro:stereo_camera_macro parent="base_link">
     <origin xyz="0 0 0" rpy="0 0 0"/>

Commit message: flipped imu

File: urdf/stereo_camera.urdf.xacro (robot description, xacro)
@@ -56,4 +56,11 @@
     <origin xyz="0 0 0" rpy="0 0 0"/>
   </xacro:stereo_camera_macro>
+  <link name="imu_link"/>
+  <joint name="imu_joint" type="fixed">
+    <parent link="base_link"/>
+    <child link="imu_link"/>
+    <!-- If IMU is rotated 180 deg around X -->
+    <origin xyz="0 0 0" rpy="0 0 3.14159"/>
+  </joint>
   <!-- Ros2 gpio controllers -->
   <!-- <ros2_control name="ros2_control" type="system">

Commit message: mostly obstacle detection changes

File: urdf/stereo_camera.urdf.xacro (robot description, xacro)
@@ -39,7 +39,7 @@
     <link name="imu_link"/>
     <joint name="imu_joint" type="fixed">
-      <parent link="camera_link"/>
+      <parent link="base_link"/>
       <child link="imu_link"/>
-      <origin xyz="0 0 0" rpy="0 0 0"/>
+      <origin xyz="0 0 0" rpy="0 0 3.14159"/>
     </joint>
     <!-- Mount to parent -->
@@ -56,11 +56,4 @@
     <origin xyz="0 0 0" rpy="0 0 0"/>
   </xacro:stereo_camera_macro>
-  <link name="imu_link"/>
-  <joint name="imu_joint" type="fixed">
-    <parent link="base_link"/>
-    <child link="imu_link"/>
-    <!-- If IMU is rotated 180 deg around X -->
-    <origin xyz="0 0 0" rpy="0 0 3.14159"/>
-  </joint>
   <!-- Ros2 gpio controllers -->
   <!-- <ros2_control name="ros2_control" type="system">

Commit message: reincorporated depth node, started readme revision, other cleanup changes

File: urdf/stereo_camera.urdf.xacro (robot description, xacro)
@@ -27,5 +27,5 @@
       <parent link="camera_link"/>
       <child link="left_camera_optical_frame"/>
-      <origin xyz="${-baseline/2} 0 0" rpy="-1.57079632679 0 -1.57079632679"/>
+      <origin xyz="${-baseline/2} 0 0" rpy="${-M_PI / 2} 0 ${-M_PI / 2}"/> <!-- Translate from standard optical coordinate frame to ROS coordinate frame -->
     </joint>
     <!-- Right camera -->
@@ -34,5 +34,5 @@
       <parent link="camera_link"/>
       <child link="right_camera_optical_frame"/>
-      <origin xyz="${baseline/2} 0 0" rpy="-1.57079632679 0 -1.57079632679"/>
+      <origin xyz="${baseline/2} 0 0" rpy="${-M_PI / 2} 0 ${-M_PI / 2}"/>  <!-- Translate from standard optical coordinate frame to ROS coordinate frame -->
     </joint>
     <!-- IMU -->
@@ -56,16 +56,3 @@
     <origin xyz="0 0 0" rpy="0 0 0"/>
   </xacro:stereo_camera_macro>
-  <!-- Ros2 gpio controllers -->
-  <!-- <ros2_control name="ros2_control" type="system">
-      <hardware>
-          <plugin>gpio_controllers/Gpios</plugin>
-          <param name="gpio_chip_name">gpiochip0</param>
-      </hardware>
-      <gpio name="button">
-          <command_interface name="value"/>
-          <state_interface name="value"/>
-          <param name="pin">17</param>
-          <param name="direction">in</param>
-      </gpio>
-  </ros2_control> -->
 </robot>
